File: battery-voltage-current-sensor.sch (EAGLE design)
At the start: 66 parts, among them IC1 ACS758LCB-050B-PFF-T, IC3 ADS1115IDGST, T1 C8545, T2 C8545, T3 C8545, X1 MKDSN1,5/2-5,08

Commit message: connector swapped against a 4pin for a display
Parts:
- removed X1: MKDSN1,5/2-5,08, con-phoenix-508:MKDSN1,5/2-5,08
- added J1: B4B-XH-A(LF)(SN), Headers:B4B-XH-A(LF)(SN)
Connections:
- net +12V/1: no longer X1-2.KL
- net +5V/1: now also J1.3
- net GND: now also J1.4; no longer X1-1.KL
- net SCL: now also J1.2
- net SDA: now also J1.1
Changed lines of the file:
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@@
 <part name="R3" library="rcl" library_urn="urn:adsk.eagle:library:334" deviceset="R-EU_" device="R0603" package3d_urn="urn:adsk.eagle:package:23555/2" value="10k"/>
 <part name="R29" library="rcl" library_urn="urn:adsk.eagle:library:334" deviceset="R-EU_" device="R0603" package3d_urn="urn:adsk.eagle:package:23555/2" value="10k"/>
-<part name="X1" library="con-phoenix-508" library_urn="urn:adsk.eagle:library:176" deviceset="MKDSN1,5/2-5,08" device="" package3d_urn="urn:adsk.eagle:package:9630/1"/>
+<part name="J1" library="Headers" library_urn="urn:adsk.eagle:library:11687645" deviceset="B4B-XH-A(LF)(SN)" device="" package3d_urn="urn:adsk.eagle:package:19181368/7"/>
 </parts>
 <sheets>
@@
 <attribute name="VALUE" x="325.882" y="31.75" size="1.778" layer="96" rot="R90"/>
 </instance>
-<instance part="X1" gate="-1" x="114.3" y="55.88" smashed="yes">
-<attribute name="NAME" x="117.348" y="54.991" size="1.778" layer="95"/>
-<attribute name="VALUE" x="111.76" y="52.197" size="1.778" layer="96"/>
-</instance>
-<instance part="X1" gate="-2" x="114.3" y="50.8" smashed="yes">
-<attribute name="NAME" x="117.348" y="49.911" size="1.778" layer="95"/>
-<attribute name="VALUE" x="111.76" y="47.117" size="1.778" layer="96"/>
+<instance part="J1" gate="G$1" x="373.38" y="73.66" smashed="yes" rot="R180">
+<attribute name="NAME" x="376.936" y="66.294" size="1.27" layer="95" rot="R180"/>
+<attribute name="VALUE" x="376.936" y="79.756" size="1.27" layer="96" rot="R180"/>
 </instance>
 </instances>
@@
 <segment>
 <pinref part="PS1" gate="G$1" pin="-VO"/>
-<wire x1="81.28" y1="63.5" x2="109.22" y2="63.5" width="0.1524" layer="91"/>
-<wire x1="109.22" y1="63.5" x2="114.3" y2="63.5" width="0.1524" layer="91"/>
+<wire x1="81.28" y1="63.5" x2="114.3" y2="63.5" width="0.1524" layer="91"/>
 <wire x1="114.3" y1="63.5" x2="114.3" y2="66.04" width="0.1524" layer="91"/>
 <label x="119.38" y="63.5" size="1.778" layer="95"/>
-<pinref part="X1" gate="-1" pin="KL"/>
-<wire x1="111.76" y1="55.88" x2="109.22" y2="55.88" width="0.1524" layer="91"/>
-<wire x1="109.22" y1="55.88" x2="109.22" y2="63.5" width="0.1524" layer="91"/>
-<junction x="109.22" y="63.5"/>
 </segment>
 <segment>
@@
 <label x="-63.5" y="195.58" size="1.778" layer="95" rot="R180"/>
 <junction x="0" y="190.5"/>
-<wire x1="0" y1="190.5" x2="66.04" y2="190.5" width="0.1524" layer="91"/>
-<wire x1="66.04" y1="190.5" x2="66.04" y2="154.94" width="0.1524" layer="91"/>
+<wire x1="0" y1="190.5" x2="68.58" y2="190.5" width="0.1524" layer="91"/>
+<wire x1="68.58" y1="190.5" x2="68.58" y2="154.94" width="0.1524" layer="91"/>
 <pinref part="IC1" gate="G$1" pin="GND"/>
 <wire x1="15.24" y1="162.56" x2="22.86" y2="162.56" width="0.1524" layer="91"/>
@@
 <wire x1="45.72" y1="154.94" x2="45.72" y2="162.56" width="0.1524" layer="91"/>
 <junction x="40.64" y="154.94"/>
-<wire x1="66.04" y1="154.94" x2="45.72" y2="154.94" width="0.1524" layer="91"/>
+<wire x1="68.58" y1="154.94" x2="45.72" y2="154.94" width="0.1524" layer="91"/>
 <junction x="45.72" y="154.94"/>
+</segment>
+<segment>
+<pinref part="J1" gate="G$1" pin="4"/>
+<wire x1="365.76" y1="76.2" x2="360.68" y2="76.2" width="0.1524" layer="91"/>
+<wire x1="360.68" y1="76.2" x2="360.68" y2="86.36" width="0.1524" layer="91"/>
+<label x="360.68" y="86.36" size="1.778" layer="95"/>
 </segment>
 </net>
@@
 <label x="320.04" y="48.26" size="1.778" layer="95"/>
 </segment>
+<segment>
+<pinref part="J1" gate="G$1" pin="3"/>
+<wire x1="365.76" y1="73.66" x2="355.6" y2="73.66" width="0.1524" layer="91"/>
+<wire x1="355.6" y1="73.66" x2="355.6" y2="86.36" width="0.1524" layer="91"/>
+<label x="350.52" y="86.36" size="1.778" layer="95"/>
+</segment>
 </net>
 <net name="SCL" class="0">
@@
 <wire x1="314.96" y1="96.52" x2="322.58" y2="96.52" width="0.1524" layer="91"/>
 <wire x1="322.58" y1="96.52" x2="322.58" y2="104.14" width="0.1524" layer="91"/>
-<wire x1="322.58" y1="96.52" x2="335.28" y2="96.52" width="0.1524" layer="91"/>
 <junction x="322.58" y="96.52"/>
 <label x="332.74" y="96.52" size="1.778" layer="95"/>
+<wire x1="322.58" y1="96.52" x2="347.98" y2="96.52" width="0.1524" layer="91"/>
+<pinref part="J1" gate="G$1" pin="2"/>
+<wire x1="347.98" y1="96.52" x2="347.98" y2="71.12" width="0.1524" layer="91"/>
+<wire x1="347.98" y1="71.12" x2="365.76" y2="71.12" width="0.1524" layer="91"/>
 </segment>
 </net>
@@
 <wire x1="81.28" y1="60.96" x2="91.44" y2="60.96" width="0.1524" layer="91"/>
 <label x="96.52" y="55.88" size="1.778" layer="95"/>
-<pinref part="X1" gate="-2" pin="KL"/>
-<wire x1="111.76" y1="50.8" x2="91.44" y2="50.8" width="0.1524" layer="91"/>
 <wire x1="91.44" y1="50.8" x2="91.44" y2="60.96" width="0.1524" layer="91"/>
 </segment>
@@
 <wire x1="314.96" y1="58.42" x2="322.58" y2="58.42" width="0.1524" layer="91"/>
 <wire x1="322.58" y1="58.42" x2="322.58" y2="66.04" width="0.1524" layer="91"/>
-<wire x1="322.58" y1="58.42" x2="335.28" y2="58.42" width="0.1524" layer="91"/>
 <junction x="322.58" y="58.42"/>
 <label x="335.28" y="58.42" size="1.778" layer="95"/>
-</segment>
-</net>
+<pinref part="J1" gate="G$1" pin="1"/>
+<wire x1="365.76" y1="68.58" x2="365.76" y2="58.42" width="0.1524" layer="91"/>
+<wire x1="365.76" y1="58.42" x2="322.58" y2="58.42" width="0.1524" layer="91"/>
+</segment>
+</net>
